Commit message: full one leg, fixed rviz config

File: spider-description/robot.urdf (robot description, URDF)
Before this commit: robot spider-description, 3 links, 2 joints
Links:
- added link moving_frame_l_3, mass 10.0269; collision mesh filename=package://spider-description/assets/femur__limb_legnth_0_5_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; collision mesh filename=package://spider-description/assets/moving_frame_l.stl
- link moving_frame_l_2: mass 6.08677 -> 12.6662; geometry collision mesh filename=package://spider-description/assets/femur__limb_legnth_0_4_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; collision mesh filename=package://spider-description/assets/motor_holder.stl
Joints:
- removed joint 1
- removed joint 2
- added joint 1-1: type revolute, parent motor_holder, child moving_frame_l, origin xyz=0 -0.107 -0.114 rpy=-5.283e-15 6.09566e-16 -1.65806, axis 0 0 1, limit lower=-1.48353 upper=1.65806 effort=10 velocity=10
- added joint 1-2: type revolute, parent moving_frame_l, child moving_frame_l_2, origin xyz=0.229 0.113838 0.11355 rpy=1.5708 0.349066 2.18573e-15, axis 0 0 1, limit lower=-1.22173 upper=1.91986 effort=10 velocity=10
- added joint 1-3: type revolute, parent moving_frame_l_2, child moving_frame_l_3, origin xyz=0.669 0.000161803 0.22755 rpy=-3.14159 3.83374e-16 -1.0472, axis 0 0 1, limit lower=-2.61799 upper=0.523599 effort=10 velocity=10

Commit message: updated motors starting position in model

File: spider-description/robot.urdf (robot description, URDF)
Before this commit: robot spider-description, 4 links, 3 joints
Joints:
- joint 1-1: limit lower=-1.48353 upper=1.65806 effort=10 velocity=10 -> lower=0 upper=3.14159 effort=10 velocity=10; origin xyz=0 -0.107 -0.114 rpy=-5.283e-15 6.09566e-16 -1.65806 -> xyz=-2.80687e-17 -0.107 -0.114 rpy=-6.07154e-16 1.44907e-19 -3.14159
- joint 1-2: limit lower=-1.22173 upper=1.91986 effort=10 velocity=10 -> lower=-2.4869e-14 upper=3.14159 effort=10 velocity=10; origin xyz=0.229 0.113838 0.11355 rpy=1.5708 0.349066 2.18573e-15 -> xyz=0.229 0.107838 0.11355 rpy=-1.5708 1.4383e-16 -3.64292e-16
- joint 1-3: limit lower=-2.61799 upper=0.523599 effort=10 velocity=10 -> lower=0 upper=3.14159 effort=10 velocity=10; origin xyz=0.669 0.000161803 0.22755 rpy=-3.14159 3.83374e-16 -1.0472 -> xyz=-0.000161803 -0.669 -0.22755 rpy=6.87867e-17 2.6966e-15 3.14159
