Commit message: renamed spider-description to spider_description

File: spider_description/robot.urdf (robot description, URDF)
Before this commit: robot spider-description, 4 links, 3 joints
Links:
- link motor_holder: geometry collision mesh filename=package://spider_description/assets/motor_holder.stl; collision mesh filename=package://spider_description/assets/motor_model.stl
- link moving_frame_l: geometry collision mesh filename=package://spider_description/assets/motor_holder.stl; collision mesh filename=package://spider_description/assets/motor_model.stl
- link moving_frame_l_2: geometry collision mesh filename=package://spider_description/assets/femur__limb_legnth_0_4_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; collision mesh filename=package://spider_description/assets/motor_holder.stl
- link moving_frame_l_3: geometry collision mesh filename=package://spider_description/assets/femur__limb_legnth_0_5_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; collision mesh filename=package://spider_description/assets/moving_frame_l.stl
