Commit message: fixed mujoco run

File: spider_ros_control/description/urdf/spider.urdf.xacro (robot description, xacro)
@@ -2,6 +2,6 @@
 <!-- Basic differential drive mobile base -->
 <robot xmlns:xacro="http://www.ros.org/wiki/xacro" name="diffdrive_robot">
-  <xacro:arg name="use_mock_hardware" default="false" />
-  <xacro:include filename="$(find spider_description)/robot.urdf" />
+  <xacro:arg name="use_mock_hardware" default="true" />
+  <xacro:include filename="$(find spider_description)/urdf/robot.urdf" />
   <ros2_control name="Spider" type="system">
     <xacro:unless value="$(arg use_mock_hardware)">
@@ -17,7 +17,8 @@
     </hardware>
     </xacro:if>
-    <joint name="1-1">
-       <param name="leg_id">1</param>
-       <param name="motor_id">1</param>
+   <xacro:macro name="joint" params="leg_id motor_id">
+    <joint name="${leg_id}-${motor_id}">
+       <param name="leg_id">${leg_id}</param>
+       <param name="motor_id">${motor_id}</param>
        <command_interface name="position"/>
        <state_interface name="position">
@@ -25,20 +26,23 @@
        </state_interface>
     </joint>
-    <joint name="1-2">
-       <param name="leg_id">1</param>
-       <param name="motor_id">2</param>
-       <command_interface name="position"/>
-       <state_interface name="position">
-          <param name="initial_value">0</param>
-       </state_interface>
-    </joint>
-    <joint name="1-3">
-       <param name="leg_id">1</param>
-       <param name="motor_id">3</param>
-       <command_interface name="position"/>
-       <state_interface name="position">
-          <param name="initial_value">0</param>
-       </state_interface>
-    </joint>
+   </xacro:macro>
+   <xacro:joint leg_id="1" motor_id="1" />
+   <xacro:joint leg_id="1" motor_id="2" />
+   <xacro:joint leg_id="1" motor_id="3" />
+   <xacro:joint leg_id="2" motor_id="1" />
+   <xacro:joint leg_id="2" motor_id="2" />
+   <xacro:joint leg_id="2" motor_id="3" />
+   <xacro:joint leg_id="3" motor_id="1" />
+   <xacro:joint leg_id="3" motor_id="2" />
+   <xacro:joint leg_id="3" motor_id="3" />
+   <xacro:joint leg_id="4" motor_id="1" />
+   <xacro:joint leg_id="4" motor_id="2" />
+   <xacro:joint leg_id="4" motor_id="3" />
+   <xacro:joint leg_id="5" motor_id="1" />
+   <xacro:joint leg_id="5" motor_id="2" />
+   <xacro:joint leg_id="5" motor_id="3" />
+   <xacro:joint leg_id="6" motor_id="1" />
+   <xacro:joint leg_id="6" motor_id="2" />
+   <xacro:joint leg_id="6" motor_id="3" />
   </ros2_control>
 </robot>
