Commit message: broke submodules, trying to fix

File: spider_ros_control/description/urdf/spider-mujoco.urdf.xacro (robot description, xacro)
@@ -19,22 +19,36 @@
     </joint>
    </xacro:macro>
-   <xacro:joint leg_id="1" motor_id="1" />
-   <xacro:joint leg_id="1" motor_id="2" />
-   <xacro:joint leg_id="1" motor_id="3" />
-   <xacro:joint leg_id="2" motor_id="1" />
-   <xacro:joint leg_id="2" motor_id="2" />
-   <xacro:joint leg_id="2" motor_id="3" />
-   <xacro:joint leg_id="3" motor_id="1" />
-   <xacro:joint leg_id="3" motor_id="2" />
-   <xacro:joint leg_id="3" motor_id="3" />
-   <xacro:joint leg_id="4" motor_id="1" />
-   <xacro:joint leg_id="4" motor_id="2" />
-   <xacro:joint leg_id="4" motor_id="3" />
-   <xacro:joint leg_id="5" motor_id="1" />
-   <xacro:joint leg_id="5" motor_id="2" />
-   <xacro:joint leg_id="5" motor_id="3" />
-   <xacro:joint leg_id="6" motor_id="1" />
-   <xacro:joint leg_id="6" motor_id="2" />
-   <xacro:joint leg_id="6" motor_id="3" />
+   <xacro:macro name="pid_joint" params="leg_id motor_id">
+    <joint name="${leg_id}-${motor_id}">
+       <param name="leg_id">${leg_id}</param>
+       <param name="motor_id">${motor_id}</param>
+       <param name="position_kp">10000</param>
+       <param name="position_ki">1</param>
+       <param name="position_kd">10</param>
+       <param name="position_i_max">10000</param>
+       <command_interface name="position_pid"/>
+       <state_interface name="position">
+          <param name="initial_value">0</param>
+       </state_interface>
+    </joint>
+   </xacro:macro>
+   <xacro:pid_joint leg_id="1" motor_id="1" />
+   <xacro:pid_joint leg_id="1" motor_id="2" />
+   <xacro:pid_joint leg_id="1" motor_id="3" />
+   <xacro:pid_joint leg_id="2" motor_id="1" />
+   <xacro:pid_joint leg_id="2" motor_id="2" />
+   <xacro:pid_joint leg_id="2" motor_id="3" />
+   <xacro:pid_joint leg_id="3" motor_id="1" />
+   <xacro:pid_joint leg_id="3" motor_id="2" />
+   <xacro:pid_joint leg_id="3" motor_id="3" />
+   <xacro:pid_joint leg_id="4" motor_id="1" />
+   <xacro:pid_joint leg_id="4" motor_id="2" />
+   <xacro:pid_joint leg_id="4" motor_id="3" />
+   <xacro:pid_joint leg_id="5" motor_id="1" />
+   <xacro:pid_joint leg_id="5" motor_id="2" />
+   <xacro:pid_joint leg_id="5" motor_id="3" />
+   <xacro:pid_joint leg_id="6" motor_id="1" />
+   <xacro:pid_joint leg_id="6" motor_id="2" />
+   <xacro:pid_joint leg_id="6" motor_id="3" />
   </ros2_control>
 </robot>
