Commit message: a lot of unfinished work on cinematics

File: spider_description/urdf/robot.urdf (robot description, URDF)
Before this commit: robot urdf, 19 links, 18 joints
Links:
- link body_plate_deepseek: mass 47.3631 -> 0
Joints:
- joint 1-1: origin xyz=0.742681 1.2304 -0.043323 rpy=0.174533 1.92679e-15 2.35619 -> xyz=1.12766 1.03602 -0.761328 rpy=0.0137696 -0.01338 2.39649
- joint 1-2: origin xyz=0.229 0.113838 0.11355 rpy=1.5708 -1.0472 4.44089e-15 -> xyz=0.229 -0.117162 0.11355 rpy=-1.5708 -1.5708 0
- joint 1-3: origin xyz=0.669 0.000161803 0.22755 rpy=3.14159 3.33067e-15 -2.0944 -> xyz=0.669 0.000161803 -0.00045 rpy=3.60822e-15 2.2482e-15 0.0258883
- joint 2-1: origin xyz=0.702046 0.877633 0.0078812 rpy=0.124042 -0.123098 3.13394 -> xyz=1.08567 0.679726 -0.758027 rpy=0.000948136 -0.0191759 -3.13631
- joint 2-2: origin xyz=0.229 0.113838 0.11355 rpy=1.5708 -0.923627 3.38353e-15 -> xyz=0.229 -0.114162 0.11355 rpy=-1.5708 -1.5708 0
- joint 2-3: origin xyz=0.669 0.000161803 0.22755 rpy=3.14159 2.65066e-15 -2.0944 -> xyz=0.669 0.000161803 -0.00045 rpy=-6.98226e-16 1.96067e-15 -0.00052111
- joint 3-1: origin xyz=0.74911 0.424697 0.058486 rpy=3.64948e-16 -0.174533 -2.35619 -> xyz=1.13201 0.223899 -0.758437 rpy=-0.01289 -0.0142294 -2.35081
- joint 3-2: origin xyz=0.229 0.113838 0.11355 rpy=1.5708 -0.959931 8.22636e-16 -> xyz=0.229 -0.114162 0.11355 rpy=-1.5708 -1.51486 -1.39638e-14
- joint 3-3: origin xyz=0.669 0.000161803 0.22755 rpy=3.14159 2.498e-15 -2.18166 -> xyz=0.669 0.000161803 -0.00045 rpy=1.94289e-15 -6.81746e-16 -0.0244188
- joint 4-1: origin xyz=1.44966 1.22525 -0.128675 rpy=-1.55969e-15 0.174533 0.785398 -> xyz=1.8397 1.03978 -0.772862 rpy=0.01289 0.0142294 0.79078
- joint 4-2: origin xyz=0.229 0.113838 0.11355 rpy=1.5708 -1.22173 -1.62304e-15 -> xyz=0.229 -0.114162 0.11355 rpy=-1.5708 -1.56204 2.16849e-14
- joint 4-3: origin xyz=0.669 0.000161803 0.22755 rpy=3.14159 -2.77556e-17 -2.0944 -> xyz=0.669 0.000161803 -0.00045 rpy=-4.44089e-16 2.21177e-16 -0.0228203
- joint 5-1: origin xyz=1.49597 0.871556 -0.090349 rpy=-0.124042 0.123098 -0.00765412 -> xyz=1.88551 0.68395 -0.773367 rpy=-0.000948136 0.0191759 0.0052813
- joint 5-2: origin xyz=0.229 0.11596 0.11355 rpy=1.5708 -1.17077 3.56348e-17 -> xyz=0.229 -0.116283 0.11355 rpy=1.5708 -1.51387 3.14159
- joint 5-3: origin xyz=0.669 0.000161803 0.22755 rpy=-3.14159 -1.52656e-16 -2.0944 -> xyz=0.669 0.000161803 -0.00045 rpy=6.08021e-16 1.44698e-15 0.0206233
- joint 6-1: origin xyz=1.45583 0.419288 -0.0289551 rpy=-0.174533 -4.2454e-15 -0.785398 -> xyz=1.844 0.227659 -0.772092 rpy=-0.0142306 0.0128887 -0.780199
- joint 6-2: origin xyz=0.229 0.113838 0.11355 rpy=1.5708 -1.0472 -3.88578e-16 -> xyz=0.229 -0.114162 0.11355 rpy=1.5708 -1.55838 3.14159
- joint 6-3: origin xyz=0.669 0.000161803 0.22755 rpy=3.14159 7.77156e-16 -2.0944 -> xyz=0.669 0.000161803 -0.00045 rpy=3.9968e-15 -2.74347e-15 9.62585e-05

Commit message: new shorter robot model, merged stls

File: spider_description/urdf/robot.urdf (robot description, URDF)
Before this commit: robot urdf, 19 links, 18 joints
Links:
- link 1brackets: geometry collision mesh filename=package://spider_description/urdf/assets/merged/1brackets_c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; visual mesh filename=package://spider_description/urdf/assets/merged/1brackets_v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
- link 1brackets_2: geometry collision mesh filename=package://spider_description/urdf/assets/merged/1brackets_2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; visual mesh filename=package://spider_description/urdf/assets/merged/1brackets_2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
- link 1brackets_3: geometry collision mesh filename=package://spider_description/urdf/assets/merged/1brackets_3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; visual mesh filename=package://spider_description/urdf/assets/merged/1brackets_3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
- link 1brackets_4: geometry collision mesh filename=package://spider_description/urdf/assets/merged/1brackets_4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; visual mesh filename=package://spider_description/urdf/assets/merged/1brackets_4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
- link 1brackets_5: geometry collision mesh filename=package://spider_description/urdf/assets/merged/1brackets_5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; visual mesh filename=package://spider_description/urdf/assets/merged/1brackets_5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
- link 1brackets_6: geometry collision mesh filename=package://spider_description/urdf/assets/merged/1brackets_6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; visual mesh filename=package://spider_description/urdf/assets/merged/1brackets_6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
- link 2limb: mass 12.6805 -> 13.4767; geometry collision mesh filename=package://spider_description/urdf/assets/merged/2limb_colli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; visual mesh filename=package://spider_description/urdf/assets/merged/2limb_visua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
- link 2limb_2: mass 12.6805 -> 13.4767; geometry collision mesh filename=package://spider_description/urdf/assets/merged/2limb_2_col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; visual mesh filename=package://spider_description/urdf/assets/merged/2limb_2_vis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
- link 2limb_3: mass 12.6805 -> 13.4767; geometry collision mesh filename=package://spider_description/urdf/assets/merged/2limb_3_col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; visual mesh filename=package://spider_description/urdf/assets/merged/2limb_3_vis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
- link 2limb_4: mass 12.6805 -> 13.4767; geometry collision mesh filename=package://spider_description/urdf/assets/merged/2limb_4_col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; visual mesh filename=package://spider_description/urdf/assets/merged/2limb_4_vis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
- link 2limb_5: mass 12.6805 -> 13.4767; geometry collision mesh filename=package://spider_description/urdf/assets/merged/2limb_5_col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; visual mesh filename=package://spider_description/urdf/assets/merged/2limb_5_vis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
- link 2limb_6: mass 12.6805 -> 13.4767; geometry collision mesh filename=package://spider_description/urdf/assets/merged/2limb_6_col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; visual mesh filename=package://spider_description/urdf/assets/merged/2limb_6_vis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
- link 3limb: mass 13.7726 -> 10.0315; geometry collision mesh filename=package://spider_description/urdf/assets/merged/3limb_colli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; visual mesh filename=package://spider_description/urdf/assets/merged/3limb_visua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
- link 3limb_2: mass 13.7726 -> 10.0315; geometry collision mesh filename=package://spider_description/urdf/assets/merged/3limb_2_col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; visual mesh filename=package://spider_description/urdf/assets/merged/3limb_2_vis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
- link 3limb_3: mass 13.7726 -> 10.0315; geometry collision mesh filename=package://spider_description/urdf/assets/merged/3limb_3_col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; visual mesh filename=package://spider_description/urdf/assets/merged/3limb_3_vis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
- link 3limb_4: mass 13.7726 -> 10.0315; geometry collision mesh filename=package://spider_description/urdf/assets/merged/3limb_4_col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; visual mesh filename=package://spider_description/urdf/assets/merged/3limb_4_vis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
- link 3limb_5: mass 13.7726 -> 10.0315; geometry collision mesh filename=package://spider_description/urdf/assets/merged/3limb_5_col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; visual mesh filename=package://spider_description/urdf/assets/merged/3limb_5_vis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
- link 3limb_6: mass 13.7726 -> 10.0315; geometry collision mesh filename=package://spider_description/urdf/assets/merged/3limb_6_col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; visual mesh filename=package://spider_description/urdf/assets/merged/3limb_6_vis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
- link body_plate_deepseek: mass 0 -> 47.3631; geometry collision mesh filename=package://spider_description/urdf/assets/merged/body_plate_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; visual mesh filename=package://spider_description/urdf/assets/merged/body_plate_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
Joints:
- joint 4-2: origin xyz=0.229 -0.114162 0.11355 rpy=-1.5708 -1.56204 2.16849e-14 -> xyz=0.229 -0.114162 0.11355 rpy=-1.5708 -1.56204 2.08928e-14
